File: PCB/PCB.brd (EAGLE design)
At the start: 100.9 x 87.3 mm, 43 parts, among them Q1 11.0592MHz

Commit message: Added adithya's files after verification
Parts:
- added PLED: (no value), led:LED5MM
- C4: value 10nF -> 0.1uF
- R1, R10, R11, R6, R7, R8: value (none) -> 10k
- R12, R17, R5: value (none) -> 1k
- R13, R14, R15, R2, R3, R4: value (none) -> 4.7k
- R9: value (none) -> 2.7k
- moved R16 87.5 mm to (47.6, 57.1), turned to 270 degrees
- moved R14 51.1 mm to (126.4, 24.8), turned to 90 degrees
- moved R17 47.1 mm to (69.2, 14.0), turned to 0 degrees
- moved R13 16.0 mm to (121.3, 75.6)
- moved KEYPAD 11.3 mm to (53.3, 71.8)
- moved R15 2.54 mm to (128.9, 24.8)
- moved R10 1.91 mm to (107.3, 40.6)
- moved RESET 1.42 mm to (78.1, 81.3)
- turned R12 to 270 degrees
Connections:
- removed net 555_O/P: 555_TIMER.3, R12.P$2
- new net N$15: PLED.A, R17.P$1
- net +10V: now also R14.P$1; no longer R15.P$1, R8.P$1
- net +5V: now also R17.P$2; no longer CD4029_1.10, CD4029_1.9, CD4029_2.10, CD4029_2.9
- net -10V: now also R8.P$1
- net A2: now also CD4029_2.14; no longer CD4029_2.11
- net A3: now also CD4029_2.11; no longer CD4029_2.14
- net CLK: now also 555_TIMER.3; no longer R12.P$1, R13.P$2
- net GND: now also CD4029_1.10, CD4029_1.9, CD4029_2.10, CD4029_2.9, PLED.K, R12.P$2, R16.P$1; no longer R14.P$1, R17.P$1
- net IOUT2: now also R15.P$2; no longer R16.P$2
- net N$11: now also R13.P$2; no longer R14.P$2
- net N$12: now also R14.P$2; no longer R15.P$2
- net N$33: now also R16.P$2; no longer R17.P$2
- net OUTPUT: now also R12.P$1, R15.P$1; no longer R16.P$1
Routing:
- net CLK: track 130.2 -> 103.2 mm, vias 2 -> 1
- net 555_O/P: track 21.5 -> 0.00 mm
- net +5V: track 238.7 -> 218.2 mm
- net P1.6: track 8.89 -> 20.7 mm
- net P1.7: track 8.89 -> 20.7 mm
- net P1.5: track 8.89 -> 20.7 mm
- net P1.4: track 8.89 -> 20.7 mm
- net P1.3: track 8.89 -> 20.7 mm
- net P1.2: track 8.89 -> 20.7 mm
- net P1.1: track 8.89 -> 20.7 mm
- net P1.0: track 8.89 -> 20.7 mm
- net A2: track 35.7 -> 26.9 mm, vias 2 -> 1
- net OUTPUT: track 20.5 -> 29.1 mm
- net N$15: track 0.00 -> 7.77 mm
- net A3: track 26.2 -> 33.5 mm
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Other:
- board text added: "Of Technology"
- board text added: "Sardar Patel Institute"
- board text added: "TSE-2018"
- board text removed: "Alpha"

Commit message: Silkscreen, mounting holes, power/ip screw terminals
Parts:
- removed +10VSUPPLY, +5VSUPPLY, -10VSUPPLY, GND_PINS: (no value), SparkFun-Connectors:1X02
- removed PLED: (no value), led:LED5MM
- added POWER: (no value), led:LED5MM
- added X4: (no value), con-ptr500:AK500/6-H
- R17: value 1k -> 330
- moved KEYPAD 13.5 mm to (64.9, 64.8)
- moved R17 10.3 mm to (78.7, 17.8), turned to 90 degrees
- moved RESET 2.59 mm to (78.6, 78.7)
- moved R2 1.42 mm to (82.5, 17.8)
- moved R3 1.42 mm to (86.4, 17.8)
- moved C3 0.76 mm to (87.1, 80.0)
- moved R4 0.64 mm to (112.4, 33.0)
- moved R6 0.25 mm to (103.3, 8.89)
Connections:
- net +10V: now also X4.2; no longer +10VSUPPLY.2
- net +5V: now also X4.3; no longer +5VSUPPLY.2
- net -10V: now also X4.1; no longer -10VSUPPLY.2
- net GND: now also POWER.K, X4.4, X4.5, X4.6; no longer +10VSUPPLY.1, +5VSUPPLY.1, -10VSUPPLY.1, GND_PINS.1, GND_PINS.2, PLED.K
- net N$15: now also POWER.A; no longer PLED.A
Routing:
- net P1.6: track 20.7 -> 6.20 mm
- net P1.7: track 20.7 -> 6.20 mm
- net P1.5: track 20.7 -> 6.20 mm
- net P1.4: track 20.7 -> 6.20 mm
- net P1.3: track 20.7 -> 6.20 mm
- net P1.2: track 20.7 -> 6.20 mm
- net P1.1: track 20.7 -> 6.20 mm
- net P1.0: track 20.7 -> 6.20 mm
- net CLK: track 103.2 -> 115.1 mm
- net N$15: track 7.77 -> 19.1 mm
- net +10V: track 140.8 -> 151.9 mm
- net RESET: track 63.9 -> 61.6 mm
- net N$1: track 9.04 -> 10.2 mm
- net -10V: track 149.0 -> 148.0 mm
- net +5V: track 218.2 -> 217.5 mm
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Other:
- board size 100.9 x 87.3 mm -> 100.9 x 86 mm
- board text added: "+10V"
- board text added: "+5V"
- board text added: "-10V"
- board text added: "GND"
- board text removed: "Of Technology"
- board text removed: "Sardar Patel Institute"

Commit message: Final-for manufacturing
Parts:
- added C8: 10nF, rcl:C025-025X050
- added JP1, JP2, SJ1, SJ2, SJ3, SJ4, SJ5, SJ6, SJ7, SJ8: (no value), jumper:SJ
- moved TP1 2.18 mm to (125.0, 3.81)
- moved TP2 1.48 mm to (129.4, 3.81)
- moved R3 1.02 mm to (85.3, 17.8)
- moved R2 0.51 mm to (82.0, 17.8)
Connections:
- new net CD1-CLK: CD4029_1.15, SJ8.1
- new net CD2-CLK: CD4029_2.15, SJ5.1
- new net N$16: DAC0808_1.14, SJ2.1
- new net OP-555-CTRL: LM148.13, LM148.14, SJ6.1
- new net OPAMP-O/P: IC741.6, JP1.2, R12.P$1, R15.P$1, SJ3.1
- net +5V: now also JP2.2
- net 555_CONTROL: now also SJ6.2, SJ7.2; no longer LM148.13, LM148.14
- net CLK: now also SJ5.2, SJ8.2; no longer CD4029_1.15, CD4029_2.15
- net GND: now also C8.1, JP1.1, SJ1.1, SJ4.1, SJ7.1
- net N$2: now also SJ2.2; no longer DAC0808_1.14
- net N$4: now also SJ4.2
- net N$5: now also SJ1.2
- net OUTPUT: now also C8.2, SJ3.2; no longer IC741.6, R12.P$1, R15.P$1
- net RESET: now also JP2.1
Routing:
- net OPAMP-O/P: track 0.00 -> 27.9 mm
- net OUTPUT: track 29.1 -> 11.7 mm
- net +5V: track 217.5 -> 207.0 mm
- net CD1-CLK: track 0.00 -> 6.11 mm
- net OP-555-CTRL: track 0.00 -> 5.75 mm
- net 555_CONTROL: track 26.5 -> 21.3 mm
- net CD2-CLK: track 0.00 -> 3.61 mm
- net N$2: track 5.34 -> 2.50 mm
- net N$5: track 17.0 -> 19.7 mm
- net N$16: track 0.00 -> 2.34 mm
- net N$4: track 9.42 -> 11.6 mm
- net CLK: track 115.1 -> 113.2 mm
- net N$1: track 10.2 -> 11.8 mm
- net +10V: track 151.9 -> 152.9 mm
Other:
- board text added: "1 Oct, 2018"
- board text added: "Sardar Patel Institute of Technology"

Commit message: Commit since not sure if any changes are made
Parts:
- C8: value 10nF -> .1u

Commit message: During assembly - changed some values
Parts:
- C3: value 10nF -> 10u
- C6, C7: value 10nF -> .1u
- R16: value (none) -> 4.7k
- R9: value 2.7k -> 4.7k
Changed lines of the file:
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@@
 <attribute name="VALUE" x="67.691" y="23.749" size="1.27" layer="27" ratio="10" rot="R180"/>
 </element>
-<element name="C3" library="rcl" library_urn="urn:adsk.eagle:library:334" package="C025-025X050" package3d_urn="urn:adsk.eagle:package:23629/2" value="10nF" x="87.122" y="80.01" smashed="yes" rot="R270">
+<element name="C3" library="rcl" library_urn="urn:adsk.eagle:library:334" package="C025-025X050" package3d_urn="urn:adsk.eagle:package:23629/2" value="10u" x="87.122" y="80.01" smashed="yes" rot="R270">
 <attribute name="MF" value="" x="87.122" y="80.01" size="1.778" layer="27" rot="R270" display="off"/>
 <attribute name="MPN" value="" x="87.122" y="80.01" size="1.778" layer="27" rot="R270" display="off"/>
@@
 <attribute name="VALUE" x="131.699" y="38.354" size="1.27" layer="27" ratio="10" rot="R90"/>
 </element>
-<element name="C6" library="rcl" library_urn="urn:adsk.eagle:library:334" package="C025-025X050" package3d_urn="urn:adsk.eagle:package:23629/2" value="10nF" x="97.79" y="46.355" smashed="yes">
+<element name="C6" library="rcl" library_urn="urn:adsk.eagle:library:334" package="C025-025X050" package3d_urn="urn:adsk.eagle:package:23629/2" value=".1u" x="97.79" y="46.355" smashed="yes">
 <attribute name="MF" value="" x="97.79" y="46.355" size="1.778" layer="27" display="off"/>
 <attribute name="MPN" value="" x="97.79" y="46.355" size="1.778" layer="27" display="off"/>
@@
 <attribute name="VALUE" x="129.921" y="24.765" size="0.6096" layer="27" font="vector" ratio="20" rot="R90" align="top-center"/>
 </element>
-<element name="R16" library="SparkFun-Resistors" library_urn="urn:adsk.eagle:library:532" package="AXIAL-0.3" package3d_urn="urn:adsk.eagle:package:39658/1" value=" " x="47.625" y="57.15" smashed="yes" rot="R270">
+<element name="R16" library="SparkFun-Resistors" library_urn="urn:adsk.eagle:library:532" package="AXIAL-0.3" package3d_urn="urn:adsk.eagle:package:39658/1" value="4.7k" x="47.625" y="57.15" smashed="yes" rot="R270">
 <attribute name="MF" value="" x="47.625" y="57.15" size="1.778" layer="27" rot="R270" display="off"/>
 <attribute name="MPN" value="" x="47.625" y="57.15" size="1.778" layer="27" rot="R270" display="off"/>
@@
 <attribute name="VALUE" x="122.301" y="24.765" size="0.6096" layer="27" font="vector" ratio="20" rot="R90" align="top-center"/>
 </element>
-<element name="R9" library="SparkFun-Resistors" library_urn="urn:adsk.eagle:library:532" package="AXIAL-0.3" package3d_urn="urn:adsk.eagle:package:39658/1" value="2.7k" x="118.745" y="24.765" smashed="yes" rot="R270">
+<element name="R9" library="SparkFun-Resistors" library_urn="urn:adsk.eagle:library:532" package="AXIAL-0.3" package3d_urn="urn:adsk.eagle:package:39658/1" value="4.7k" x="118.745" y="24.765" smashed="yes" rot="R270">
 <attribute name="MF" value="" x="118.745" y="24.765" size="1.778" layer="27" rot="R270" display="off"/>
 <attribute name="MPN" value="" x="118.745" y="24.765" size="1.778" layer="27" rot="R270" display="off"/>
@@
 <attribute name="VALUE" x="129.413" y="3.81" size="0.0254" layer="27" rot="R270"/>
 </element>
-<element name="C7" library="rcl" library_urn="urn:adsk.eagle:library:334" package="C025-025X050" package3d_urn="urn:adsk.eagle:package:23629/2" value="10nF" x="90.17" y="80.01" smashed="yes" rot="R270">
+<element name="C7" library="rcl" library_urn="urn:adsk.eagle:library:334" package="C025-025X050" package3d_urn="urn:adsk.eagle:package:23629/2" value=".1u" x="90.17" y="80.01" smashed="yes" rot="R270">
 <attribute name="MF" value="" x="90.17" y="80.01" size="1.778" layer="27" rot="R270" display="off"/>
 <attribute name="MPN" value="" x="90.17" y="80.01" size="1.778" layer="27" rot="R270" display="off"/>
